File: pcb-design/pcb-design.kicad_pcb (KiCad board)
At the start: 2 copper layers, 18 parts, among them J1 Screw_Terminal_Motor, J2 Screw_Terminal_Heater, J3 Screw_Terminal_Heater, J4 Screw_Terminal_AC_Power, J5 Screw_Terminal_DC_Power, K1 ADW11, Q1 IRF3205, Q2 IRF3205, Q3 IRF3205, U1 DS18B20, U2 YAAJ_DCDC_StepDown_LM2596, U3 A4988_STEPPER_MOTOR_DRIVER_CA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

Commit message: design
Parts:
- added C1: C 16V 100nF, Capacitor_THT:C_Disc_D7.5mm_W5.0mm_P7.50mm, F.Cu at (21.0, 36.8)
- added U4: ESP32-DEVKIT-V1, local_lib:MODULE_ESP32_DEVKIT_V1, F.Cu at (50.3, 160.1)
- J1: footprint TerminalBlock_4Ucon:TerminalBlock_4Ucon_1x02_P3.50mm_Horizontal -> TerminalBlock:TerminalBlock_Altech_AK300-4_P5.00mm
- J2, J4, J5: footprint TerminalBlock_4Ucon:TerminalBlock_4Ucon_1x02_P3.50mm_Horizontal -> TerminalBlock:TerminalBlock_Altech_AK300-2_P5.00mm
- J3: value Screw_Terminal_Heater -> Screw_Terminal_Bubler; footprint TerminalBlock_4Ucon:TerminalBlock_4Ucon_1x02_P3.50mm_Horizontal -> TerminalBlock:TerminalBlock_Altech_AK300-2_P5.00mm
- R1, R2, R3, R4, R5, R6: footprint Resistor_THT:R_Axial_DIN0207_L6.3mm_D2.5mm_P2.54mm_Vertical -> Resistor_THT:R_Axial_DIN0207_L6.3mm_D2.5mm_P7.62mm_Horizontal
- U1: value DS18B20 -> DS18B20 - temperature sensor
- U3: value A4988_STEPPER_MOTOR_DRIVER_CARRIER -> TMC2209_SILENTSTEPSTICK; footprint local_lib:A4988_motor -> local_lib:MODULE_TMC2209_SILENTSTEPSTICK
- moved J1 138.1 mm to (195.9, 156.8)
- moved J5 136.1 mm to (25.4, 24.1), turned to 180 degrees
- moved U3 134.5 mm to (203.8, 135.9), turned to 90 degrees
- moved J4 122.2 mm to (266.7, 19.2)
- moved J3 115.3 mm to (266.3, 34.4)
- moved U1 111.6 mm to (33.6, 132.7)
- moved K1 92.5 mm to (251.1, 29.0)
- moved Q1 88.9 mm to (95.8, 39.1)
- moved Q3 82.4 mm to (235.1, 40.2)
- moved R1 81.2 mm to (95.0, 20.6)
- moved R6 74.3 mm to (237.4, 22.6)
- moved R4 65.2 mm to (238.3, 51.6)
- moved R5 64.7 mm to (109.0, 47.1)
- moved Q2 64.6 mm to (120.5, 22.1)
- moved R3 63.0 mm to (110.4, 38.4)
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Connections:
- U3 pad 10: +12V -> /signal_step
- U3 pad 11: Net-(J1-Pin_2) -> unconnected-(U3-PDN-Pad11)
- U3 pad 12: Net-(J1-Pin_1) -> unconnected-(U3-UART-Pad12)
- U3 pad 13: Net-(J1-Pin_3) -> unconnected-(U3-SPRD-Pad13)
- U3 pad 14: Net-(J1-Pin_4) -> unconnected-(U3-MS2-Pad14)
- U3 pad 15: GND -> unconnected-(U3-MS1-Pad15)
- U3 pad 16: +12V -> GND
- U3 pad 3: GND -> Net-(J1-Pin_3)
- U3 pad 4: GND -> Net-(J1-Pin_1)
- U3 pad 5: /signal_reset -> Net-(J1-Pin_2)
- U3 pad 6: /^signal_sleep -> Net-(J1-Pin_4)
- U3 pad 7: /signal_step -> GND
- U3 pad 8: /signal_dir -> +12V
- U3 pad 9: GND -> /signal_dir

Commit message: divided pcs
Parts:
- removed K1: ADW11, Relay_THT:Relay_1P1T_NO_10x24x18.8mm_Panasonic_ADW11xxxxW_THT
- removed Q3: IRF3205, Package_TO_SOT_THT:TO-220-3_Vertical
- removed R4, R5, R6: 10k, Resistor_THT:R_Axial_DIN0207_L6.3mm_D2.5mm_P7.62mm_Horizontal
- added J6: rj45_main, Connector_RJ:RJ45_OST_PJ012-8P8CX_Vertical, F.Cu at (135.9, 138.4)
- added J7: RJ45, Connector_RJ:RJ45_OST_PJ012-8P8CX_Vertical, F.Cu at (222.2, 125.7)
- added J8: Screw_Terminal_Bubler, TerminalBlock:TerminalBlock_Altech_AK300-2_P5.00mm, F.Cu at (251.0, 27.2)
- added J9: Power_transfer_cable_slave, TerminalBlock:TerminalBlock_Altech_AK300-2_P5.00mm, F.Cu at (218.4, 144.9)
- added K2: ADW11, Relay_THT:Relay_1P1T_NO_10x24x18.8mm_Panasonic_ADW11xxxxW_THT, F.Cu at (238.1, 22.6)
- added Q4: MT3203_heater, Package_TO_SOT_THT:TO-220-3_Vertical, F.Cu at (101.6, 33.0)
- added Q5: MT3203_heater, Package_TO_SOT_THT:TO-220-3_Vertical, F.Cu at (101.6, 45.7)
- added R10: 10k, Resistor_THT:R_Axial_DIN0207_L6.3mm_D2.5mm_P7.62mm_Horizontal, F.Cu at (261.6, 45.7)
- added R7: 4k7, Resistor_THT:R_Axial_DIN0207_L6.3mm_D2.5mm_P7.62mm_Horizontal, F.Cu at (265.4, 144.8)
- added R8: 10k, Resistor_THT:R_Axial_DIN0207_L6.3mm_D2.5mm_P7.62mm_Horizontal, F.Cu at (249.2, 36.2)
- added R9: 10k, Resistor_THT:R_Axial_DIN0207_L6.3mm_D2.5mm_P7.62mm_Horizontal, F.Cu at (249.2, 40.2)
- J3: value Screw_Terminal_Bubler -> Screw_Terminal_AC_Power
- J4: value Screw_Terminal_AC_Power -> Power_transfer_cable_main
- Q1: value IRF3205 -> IRF3205_heater
- Q2: value IRF3205 -> IRF3205_bubler
- R1: value 10k -> 2k2
- R2: value 10k -> 100
- U1: value DS18B20 - temperature sensor -> temperature sensor
- U2: value YAAJ_DCDC_StepDown_LM2596 -> step_down_converter
- U3: value TMC2209_SILENTSTEPSTICK -> TMC2209_stepper_driver
- moved U1 203.0 mm to (236.0, 147.3)
- moved J2 186.0 mm to (264.2, 132.2), turned to -90 degrees
- moved J4 161.4 mm to (142.2, 121.9), turned to 90 degrees
- moved Q2 142.0 mm to (261.6, 38.1)
- moved J1 84.6 mm to (264.2, 106.8), turned to -90 degrees
- moved U3 40.8 mm to (242.6, 123.2), turned to 180 degrees
- moved R1 39.6 mm to (133.3, 30.5)
- moved Q1 27.6 mm to (121.9, 30.5), turned to -90 degrees
- moved R3 27.3 mm to (130.8, 20.3)
- moved J3 24.8 mm to (253.9, 55.9), turned to 180 degrees
- moved R2 20.8 mm to (111.8, 20.3)
- moved U4 18.6 mm to (56.2, 177.8)
- moved U2 3.59 mm to (36.8, 48.3)
Connections:
- J2 pad 2: GND -> +12V
- J3 pad 2: Net-(J3-Pin_2) -> AC
- J4 pad 1: Earth -> Net-(J4-Pin_1)
- J4 pad 2: AC -> Net-(J4-Pin_2)
- Q2 pad 1: Net-(Q2-G) -> /Bubler driver circuit/^signal_bubler_enable
- Q2 pad 2: Net-(J2-Pin_1) -> Net-(Q2-D)
- R2 pad 2: Net-(Q2-G) -> Net-(Q4-G)
- U1 pad 2: +3.3V -> /signal_temp_probe
- U1 pad 3: GND -> +3.3V
- U3 pad 10: /signal_step -> unconnected-(U3-STEP-Pad10)
- U3 pad 12: unconnected-(U3-UART-Pad12) -> signal_uart_rx
- U3 pad 13: unconnected-(U3-SPRD-Pad13) -> signal_uart_tx
- U3 pad 9: /signal_dir -> unconnected-(U3-DIR-Pad9)
- U4 pad 19: +3.3V -> /signal_temp_probe
- U4 pad 20: /signal_dir -> unconnected-(U4-D35-Pad20)
- U4 pad 21: unconnected-(U4-D32-Pad21) -> signal_uart_rx
- U4 pad 22: /signal_step -> unconnected-(U4-D33-Pad22)
- U4 pad 25: unconnected-(U4-D27-Pad25) -> signal_uart_tx
- U4 pad 4: /^signal_heater -> unconnected-(U4-D2-Pad4)
